Commit message: floting joints

File: src/smart_knife/knife/urdf/knife.urdf (robot description, URDF)
Before this commit: robot knife_description, 4 links, 3 joints
Links:
- removed link base_link_1
- removed link base_link_2
- removed link sensortile_imu
- added link knife_base
Joints:
- removed joint joint_knife_x
- removed joint joint_knife_y
- removed joint joint_knife_z
- added joint joint_knife: type floating, parent knife_base, child knife_link, origin xyz=0 0 0 rpy=0 0 0
